Commit message: update testkit

File: robot/visual/testkit.xacro (robot description, xacro)
@@ -5,5 +5,5 @@
             <origin rpy="1.571 0 0" xyz="0.0 0.0 0.0" />
             <geometry>
-                <mesh filename="package://testkit/meshes/Transport_TestKit_Plate.stl" scale="0.001 0.001 0.001"/>
+                <mesh filename="package://testkit/meshes/Transport_TestKit.stl" scale="0.001 0.001 0.001"/>
             </geometry>
         </visual>
@@ -46,5 +46,5 @@
         <limit effort="1000.0" lower="0.0" upper="6.28" velocity="0.5" />
         <axis xyz="0 0 1" />
-        <origin xyz="0 0.07 -0.14" rpy="-1.571 0 0"/>
+        <origin xyz="0.125 -0.09 0.044" rpy="-1.571 0 0"/>
     </joint>
     <joint name="link_0_to_link_2" type="continuous">
@@ -53,5 +53,5 @@
         <limit effort="1000.0" lower="0.0" upper="6.28" velocity="0.5" />
         <axis xyz="0 0 1" />
-        <origin xyz="0 -0.6 -0.14" rpy="1.571 0 0"/>
+        <origin xyz="0.125 -0.78 0.044" rpy="1.571 0 0"/>
     </joint>
     <joint name="link_0_to_link_3" type="continuous">
@@ -60,5 +60,5 @@
         <limit effort="1000.0" lower="0.0" upper="6.28" velocity="0.5" />
         <axis xyz="0 0 1" />
-        <origin xyz="0.69 0.07 -0.14" rpy="-1.571 0 0"/>
+        <origin xyz="0.74 -0.09 0.044" rpy="-1.571 0 0"/>
     </joint>
     <joint name="link_0_to_link_4" type="continuous">
@@ -67,5 +67,5 @@
         <limit effort="1000.0" lower="0.0" upper="6.28" velocity="0.5" />
         <axis xyz="0 0 1" />
-        <origin xyz="0.69 -0.6 -0.14" rpy="1.571 0 0"/>
+        <origin xyz="0.74 -0.78 0.044" rpy="1.571 0 0"/>
     </joint>
 </robot>

Commit message: Update testkit.xacro

File: robot/visual/testkit.xacro (robot description, xacro)
@@ -1,7 +1,17 @@
 <?xml version="1.0"?>
 <robot xmlns:xacro="http://www.ros.org/wiki/xacro" name="example">
+    <xacro:property name="x_offset" value="-0.4325" />
+    <xacro:property name="y_offset" value="0.435" />
+    <xacro:property name="z_offset" value="-0.19" />
+    <link name="footprint_link">
+        <visual>
+            <origin rpy="0 0 0" xyz="0.0 0.0 0.0" />
+            <geometry>
+            </geometry>
+        </visual>
+    </link>
     <link name="link_0">
         <visual>
-            <origin rpy="1.571 0 0" xyz="0.0 0.0 0.0" />
+            <origin rpy="1.571 0 0" xyz="-0.4325 0.435 -0.19" />
             <geometry>
                 <mesh filename="package://testkit/meshes/Transport_TestKit.stl" scale="0.001 0.001 0.001"/>
@@ -41,4 +51,9 @@
         </visual>
     </link>
+    <joint name="footprint_to_link_0" type="fixed">
+        <parent link="footprint_link" />
+        <child link="link_0" />
+        <origin xyz="0 0 0.19" rpy="0 0 0"/>
+    </joint>
     <joint name="link_0_to_link_1" type="continuous">
         <parent link="link_0" />
@@ -46,5 +61,5 @@
         <limit effort="1000.0" lower="0.0" upper="6.28" velocity="0.5" />
         <axis xyz="0 0 1" />
-        <origin xyz="0.125 -0.09 0.044" rpy="-1.571 0 0"/>
+        <origin xyz="${x_offset+0.125} ${y_offset-0.09} ${z_offset+0.044}" rpy="-1.571 0 0"/>
     </joint>
     <joint name="link_0_to_link_2" type="continuous">
@@ -53,5 +68,5 @@
         <limit effort="1000.0" lower="0.0" upper="6.28" velocity="0.5" />
         <axis xyz="0 0 1" />
-        <origin xyz="0.125 -0.78 0.044" rpy="1.571 0 0"/>
+        <origin xyz="${x_offset+0.125} ${y_offset-0.78} ${z_offset+0.044}" rpy="1.571 0 0"/>
     </joint>
     <joint name="link_0_to_link_3" type="continuous">
@@ -60,5 +75,5 @@
         <limit effort="1000.0" lower="0.0" upper="6.28" velocity="0.5" />
         <axis xyz="0 0 1" />
-        <origin xyz="0.74 -0.09 0.044" rpy="-1.571 0 0"/>
+        <origin xyz="${x_offset+0.74} ${y_offset-0.09} ${z_offset+0.044}" rpy="-1.571 0 0"/>
     </joint>
     <joint name="link_0_to_link_4" type="continuous">
@@ -67,5 +82,5 @@
         <limit effort="1000.0" lower="0.0" upper="6.28" velocity="0.5" />
         <axis xyz="0 0 1" />
-        <origin xyz="0.74 -0.78 0.044" rpy="1.571 0 0"/>
+        <origin xyz="${x_offset+0.74} ${y_offset-0.78} ${z_offset+0.044}" rpy="1.571 0 0"/>
     </joint>
 </robot>
